File: radio/radio.kicad_pcb (KiCad board)
At the start: 2 copper layers, 100 x 70 mm, 19 parts, among them J1 Conn_01x04, J2 ESP32_LEFT, J3 ESP32_RIGHT, J4 FM_SPEAKERS, J5 RADIO_MIC, J6 ANTENNA_VHF, J7 BATTERY_18650, J8 POWER_SWITCH, SW1 ROTARY_ENCODER, SW2 SW_Push, SW3 SW_Push, SW4 SW_Push, U2 SA828-VHF, U3 RDA5807M-FM, U4 PAM8403-FM-AMP, U5 TP4056_CHARGER, U6 5V_BOOST, U7 3V3_REGULATOR

Commit message: pcb_v1
Parts:
- removed C1: 100nF, Capacitor_THT:C_Disc_D5.0mm_W2.5mm_P5.00mm
- removed U4: PAM8403-FM-AMP, Package_SO:SOIC-16_3.9x9.9mm_P1.27mm
- added PAM8403_LEFT1: Conn_01x04, Connector_PinHeader_2.54mm:PinHeader_1x04_P2.54mm_Vertical, F.Cu at (180.0, 95.0)
- added PAM8403_RIGHT1: Conn_01x04, Connector_PinHeader_2.54mm:PinHeader_1x04_P2.54mm_Vertical, F.Cu at (194.0, 95.0)
- moved J4 5.10 mm to (197.0, 109.4)
Routing:
- net GND: track 0.00 -> 341.3 mm, vias 0 -> 1
- net +5V: track 0.00 -> 121.7 mm, vias 0 -> 1
- net +3V3: track 0.00 -> 109.8 mm, vias 0 -> 2
- net /RADIO_PTT: track 0.00 -> 87.5 mm, vias 0 -> 1
- net /RADIO_CS: track 0.00 -> 65.0 mm
- net /BAT+: track 0.00 -> 57.8 mm
- net /VHF_ANT: track 0.00 -> 45.3 mm
- net /RADIO_TX: track 0.00 -> 37.7 mm, vias 0 -> 3
- net /RADIO_RX: track 0.00 -> 36.5 mm, vias 0 -> 1
- net /RADIO_SPKEN: track 0.00 -> 34.5 mm
- net /OLED_SDA: track 0.00 -> 30.9 mm
- net /OLED_SCL: track 0.00 -> 30.9 mm, vias 0 -> 1
- net /ENC_A: track 0.00 -> 30.2 mm
- net /ENC_B: track 0.00 -> 29.1 mm
- net /BACK_BTN: track 0.00 -> 29.0 mm
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